File: controller/controller.kicad_pcb (KiCad board)
At the start: 4 copper layers, 75 x 62.1 mm, 14 parts, among them SW10 SW_Push, SW11 SW_Push, SW2 SW_SPDT, SW3 SW_SPDT, SW4 SW_SPDT, SW5 SW_SPDT, SW8 SW_Push, SW9 SW_Push, U1 Sparkfun_Pro_Micro

Commit message: Fix ERC errors, redraw schematic, add project-local KiCad libraries
Schematic (rev 0.2, KiCad 9 file format):
- Add PWR_FLAG on +5V and GND at the Pro Micro, which resolves the two
  "Input Power pin not driven by any Output Power pins" ERC errors.
- Redraw the SparkFun Pro Micro symbol with power pins on top, ground pins
  at the bottom and the eight used inputs on the left.
- Replace the fan-out wires with net labels MODE1..4 and BTN1..4, group
  each toggle/button pair as a channel, add design notes, an A4 sheet and
  a filled-in title block.
- Renumber designators per channel (toggles SW1/3/5/7, buttons SW2/4/6/8).
  References are hidden on the silkscreen, so the fabricated board is not
  affected. Connectivity is unchanged; verified by comparing netlists.

Libraries:
- Move the embedded Pro Micro symbol, Pro Micro footprint, custom AEDIKO
  SPDT toggle footprint and logo footprint into controller/lib and register
  them in project sym-lib-table and fp-lib-table. This resolves the six
  "library not in the current configuration" ERC warnings and makes the
  project self-contained.
- The exported toggle footprint had its keep-out zone at board coordinates
  (KiCad export bug); moved to the footprint origin so DRC no longer
  reports a library mismatch.

PCB:
- Point footprints at the new library ids, rename references and nets to
  match the schematic, mark mounting holes H1..H4 and the logo as
  board-only. DRC with --schematic-parity reports 0 parity issues.

README: regenerate the schematic image and describe the labels and
libraries.

Co-Authored-By: Claude Fable 5.1 <noreply@anthropic.com>
Parts:
- G1: renamed from G***; footprint LOGO -> controller:Logo
- SW1: renamed from SW4; value SW_SPDT -> AEDIKO SPDT on-on micro toggle; footprint AEDIKO-Micro-Toggle-Switch-3-Pin-SPDT-on-on:spdt-on-on-micro-toggle-switch -> controller:SW_Toggle_SPDT_AEDIKO_Micro
- SW2: renamed from SW11; value SW_Push -> Cherry MX 1.5u
- SW3: value SW_SPDT -> AEDIKO SPDT on-on micro toggle; footprint AEDIKO-Micro-Toggle-Switch-3-Pin-SPDT-on-on:spdt-on-on-micro-toggle-switch -> controller:SW_Toggle_SPDT_AEDIKO_Micro
- SW4: renamed from SW10; value SW_Push -> Cherry MX 1.5u
- SW5: renamed from SW2; value SW_SPDT -> AEDIKO SPDT on-on micro toggle; footprint AEDIKO-Micro-Toggle-Switch-3-Pin-SPDT-on-on:spdt-on-on-micro-toggle-switch -> controller:SW_Toggle_SPDT_AEDIKO_Micro
- SW6: renamed from SW8; value SW_Push -> Cherry MX 1.5u
- SW7: renamed from SW5; value SW_SPDT -> AEDIKO SPDT on-on micro toggle; footprint AEDIKO-Micro-Toggle-Switch-3-Pin-SPDT-on-on:spdt-on-on-micro-toggle-switch -> controller:SW_Toggle_SPDT_AEDIKO_Micro
- SW8: renamed from SW9; value SW_Push -> Cherry MX 1.5u
- U1: value Sparkfun_Pro_Micro -> SparkFun Pro Micro; footprint Arduino:Sparkfun_Pro_Micro -> controller:SparkFun_Pro_Micro
- renumbered REF** to H1, REF** to H2, REF** to H3, REF** to H4
Connections:
- net Net-(SW2-B) renamed /MODE3
- net Net-(SW3-B) renamed /MODE2
- net Net-(SW4-B) renamed /MODE1
- net Net-(SW5-B) renamed /MODE4
- net Net-(U1-D7) renamed /BTN3
- net Net-(U1-D8/A8) renamed /BTN4
- net Net-(U1-~D3) renamed /BTN1
- net Net-(U1-~D5) renamed /BTN2
